File: KiCad Files/Led_Cube_BaseControler/Led_Cube_BaseControler 1mm wires.kicad_pcb (KiCad board)
At the start: 2 copper layers, 180.3 x 96.5 mm, 86 parts, among them J1 Arduino_Connection_Pins, J10 Row_08, J11 To_Next_board, J3 Row_01, J4 Row_02, J5 Row_03, J6 Row_04, J7 Row_05, J8 Row_06, J9 Row_07, U1 74HC595, U2 74HC595, U3 74HC595, U4 74HC595, U5 74HC595, U6 74HC595, U7 74HC595, U8 74HC595

Commit message: pcb design new versions, request letters
Connections:
- R17 pad 1: Net-(U2-QA) -> Net-(J1-Pin_6)
- U2 pad 15: Net-(U2-QA) -> Net-(J1-Pin_6)
- U3 pad 16: Net-(J1-Pin_6) -> Net-(J1-Pin_1)
Routing:
- net Net-(U2-QA): track 49.7 -> 0.00 mm
- net Net-(J1-Pin_6): track 156.1 -> 194.2 mm
- net Net-(J1-Pin_1): track 77.4 -> 88.9 mm
